File: boards/rev_A/epoch_revA.sch (EAGLE design)
At the start: 16 parts, among them J1 Qwiic Right Angle, J2 1140084168, J3 105450-0101, J4 FTSH-105-01-F-DV-K-TRJ, U1 ESP32-WROOM-32D, U2 ICM-20948, U3 NEO-M8Q, U4 USBLC6-2P6, U5 MCP73811T-420I/OT, U6 TPS613221ADBVR

Commit message: started defining board outline
Parts:
- added FD1, FD2: FIDUCIAL1X2, SparkFun-Aesthetics:FIDUCIAL1X2
Connections:
- new net N$2: R37.2, R39.2, R40.2
- new net SD_CLK: U1.IO14
- new net SD_CMD: U1.IO15
- new net SD_D0: U1.IO2
- new net SD_D1: U1.IO4
- new net SD_D2: U1.IO12
- new net SD_D3: U1.IO13
- net +3V3: now also U1.3V3, U1.EN; no longer R37.2, R39.2, R40.2
- net GND: now also U1.GND
Other:
- note added: "Bluetooth MCU"
- note removed: "FPGA USB"

Commit message: working on pin connections
Parts:
- removed C57: 10uF, Resistor_Capacitor:CC0402JRNPO9BN100
- removed R37, R39, R40: 10K, Resistor_Capacitor:RC0402JR-070RL
Connections:
- removed net FPGA_CS: R37.1
- removed net HOLD: R40.1
- removed net N$2: R37.2, R39.2, R40.2
- removed net VCC: C57.1
- removed net WP: R39.1
- new net I2C_SCL: U1.IO22
- new net I2C_SDA: U1.IO23
- new net LED_CTRL: U1.IO19
- new net RXD: U1.RXD0
- new net SPI_CS: U1.IO21
- new net SPI_MISO: U1.IO16
- new net SPI_MOSI: U1.IO17
- new net SPI_SCK: U1.IO18
- new net STRAP_1: U1.IO0
- new net STRAP_4: U1.IO5
- new net TXD: U1.TXD0
- net GND: no longer C57.2
Changed lines of the file:
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@@
 <part name="GND58" library="supply1" library_urn="urn:adsk.eagle:library:371" deviceset="GND" device=""/>
 <part name="P+9" library="supply1" library_urn="urn:adsk.eagle:library:371" deviceset="VCC" device=""/>
-<part name="R39" library="Resistor_Capacitor" library_urn="urn:adsk.eagle:library:11396451" deviceset="RC0402JR-070RL" device="" package3d_urn="urn:adsk.eagle:package:10872901/3" value="10K">
-<attribute name="DIGIKEY_PART_NUMBER" value=""/>
-<attribute name="MPN" value="AC0402FR-1310KL"/>
-</part>
-<part name="R40" library="Resistor_Capacitor" library_urn="urn:adsk.eagle:library:11396451" deviceset="RC0402JR-070RL" device="" package3d_urn="urn:adsk.eagle:package:10872901/3" value="10K">
-<attribute name="DIGIKEY_PART_NUMBER" value=""/>
-<attribute name="MPN" value="AC0402FR-1310KL"/>
-</part>
-<part name="R37" library="Resistor_Capacitor" library_urn="urn:adsk.eagle:library:11396451" deviceset="RC0402JR-070RL" device="" package3d_urn="urn:adsk.eagle:package:10872901/3" value="10K">
-<attribute name="DIGIKEY_PART_NUMBER" value=""/>
-<attribute name="MPN" value="AC0402FR-1310KL"/>
-</part>
-<part name="C57" library="Resistor_Capacitor" library_urn="urn:adsk.eagle:library:11396451" deviceset="CC0402JRNPO9BN100" device="" package3d_urn="urn:adsk.eagle:package:10872910/2" value="10uF">
-<attribute name="DIGIKEY_PART_NUMBER" value=""/>
-<attribute name="MANUFACTURER" value="Murata"/>
-<attribute name="MPN" value="GRM155C80G106ME44D"/>
-</part>
 <part name="P+7" library="supply1" library_urn="urn:adsk.eagle:library:371" deviceset="VCC" device=""/>
 <part name="GND57" library="supply1" library_urn="urn:adsk.eagle:library:371" deviceset="GND" device=""/>
@@
 <attribute name="VALUE" x="101.6" y="127" size="1.778" layer="96"/>
 </instance>
-<instance part="R39" gate="G$1" x="204.47" y="137.16" smashed="yes" rot="R90">
-<attribute name="NAME" x="202.9714" y="134.62" size="1.778" layer="95" rot="R90"/>
-<attribute name="VALUE" x="207.772" y="134.62" size="1.778" layer="96" rot="R90"/>
-</instance>
-<instance part="R40" gate="G$1" x="212.09" y="137.16" smashed="yes" rot="R90">
-<attribute name="NAME" x="210.5914" y="134.62" size="1.778" layer="95" rot="R90"/>
-<attribute name="VALUE" x="215.392" y="134.62" size="1.778" layer="96" rot="R90"/>
-</instance>
-<instance part="R37" gate="G$1" x="196.85" y="137.16" smashed="yes" rot="R90">
-<attribute name="NAME" x="195.3514" y="134.62" size="1.778" layer="95" rot="R90"/>
-<attribute name="VALUE" x="200.152" y="134.62" size="1.778" layer="96" rot="R90"/>
-</instance>
-<instance part="C57" gate="G$1" x="38.1" y="128.27" smashed="yes">
-<attribute name="NAME" x="39.37" y="129.413" size="1.778" layer="95"/>
-<attribute name="VALUE" x="39.37" y="123.19" size="1.778" layer="96"/>
-</instance>
 <instance part="P+7" gate="VCC" x="38.1" y="134.62" smashed="yes">
 <attribute name="VALUE" x="35.56" y="135.89" size="1.778" layer="96"/>
@@
 <junction x="67.31" y="124.46"/>
 </segment>
-<segment>
-<pinref part="C57" gate="G$1" pin="2"/>
-<pinref part="GND57" gate="1" pin="GND"/>
-</segment>
 </net>
 <net name="FPGA_USB_P" class="1">
@@
 </segment>
 <segment>
-<pinref part="C57" gate="G$1" pin="1"/>
 <pinref part="P+7" gate="VCC" pin="VCC"/>
 <wire x1="38.1" y1="130.81" x2="38.1" y2="132.08" width="0.1524" layer="91"/>
@@
 <net name="FPGA_CS" class="0">
 <segment>
-<pinref part="R37" gate="G$1" pin="1"/>
 <wire x1="196.85" y1="130.81" x2="196.85" y2="132.08" width="0.1524" layer="91"/>
 <label x="196.85" y="130.81" size="1.27" layer="95" ratio="10" rot="R270" xref="yes"/>
@@
 <net name="WP" class="0">
 <segment>
-<pinref part="R39" gate="G$1" pin="1"/>
 <wire x1="204.47" y1="130.81" x2="204.47" y2="132.08" width="0.1524" layer="91"/>
 <label x="204.47" y="130.81" size="1.27" layer="95" ratio="10" rot="R270" xref="yes"/>
@@
 <net name="HOLD" class="0">
 <segment>
-<pinref part="R40" gate="G$1" pin="1"/>
 <wire x1="212.09" y1="130.81" x2="212.09" y2="132.08" width="0.1524" layer="91"/>
 <label x="212.09" y="130.81" size="1.27" layer="95" ratio="10" rot="R270" xref="yes"/>
@@
 <wire x1="204.47" y1="144.78" x2="204.47" y2="143.51" width="0.1524" layer="91"/>
 <wire x1="204.47" y1="143.51" x2="212.09" y2="143.51" width="0.1524" layer="91"/>
-<pinref part="R40" gate="G$1" pin="2"/>
 <wire x1="212.09" y1="143.51" x2="212.09" y2="142.24" width="0.1524" layer="91"/>
-<pinref part="R39" gate="G$1" pin="2"/>
 <wire x1="204.47" y1="143.51" x2="204.47" y2="142.24" width="0.1524" layer="91"/>
 <junction x="204.47" y="143.51"/>
-<pinref part="R37" gate="G$1" pin="2"/>
 <wire x1="196.85" y1="142.24" x2="196.85" y2="143.51" width="0.1524" layer="91"/>
 <wire x1="196.85" y1="143.51" x2="204.47" y2="143.51" width="0.1524" layer="91"/>
@@
 <pinref part="U1" gate="G$1" pin="IO12"/>
 </segment>
+<segment>
+<wire x1="129.54" y1="166.37" x2="128.27" y2="166.37" width="0.1524" layer="91"/>
+<label x="128.27" y="166.37" size="1.27" layer="95" rot="R180" xref="yes"/>
+</segment>
 </net>
 <net name="SD_D3" class="0">
@@
 <pinref part="U1" gate="G$1" pin="IO15"/>
 </segment>
+<segment>
+<wire x1="129.54" y1="157.48" x2="128.27" y2="157.48" width="0.1524" layer="91"/>
+<label x="128.27" y="157.48" size="1.27" layer="95" rot="R180" xref="yes"/>
+</segment>
 </net>
 <net name="SD_D0" class="0">
@@
 <pinref part="U1" gate="G$1" pin="IO2"/>
 </segment>
+<segment>
+<wire x1="129.54" y1="162.56" x2="128.27" y2="162.56" width="0.1524" layer="91"/>
+<label x="128.27" y="162.56" size="1.27" layer="95" rot="R180" xref="yes"/>
+</segment>
 </net>
 <net name="SD_D1" class="0">
@@
 </segment>
 </net>
+<net name="TXD" class="0">
+<segment>
+<pinref part="U1" gate="G$1" pin="TXD0"/>
+<wire x1="54.61" y1="158.75" x2="55.88" y2="158.75" width="0.1524" layer="91"/>
+<label x="54.61" y="158.75" size="1.27" layer="95" rot="R180" xref="yes"/>
+</segment>
+</net>
+<net name="RXD" class="0">
+<segment>
+<pinref part="U1" gate="G$1" pin="RXD0"/>
+<wire x1="54.61" y1="156.21" x2="55.88" y2="156.21" width="0.1524" layer="91"/>
+<label x="54.61" y="156.21" size="1.27" layer="95" rot="R180" xref="yes"/>
+</segment>
+</net>
+<net name="SPI_MISO" class="0">
+<segment>
+<wire x1="92.71" y1="156.21" x2="91.44" y2="156.21" width="0.1524" layer="91"/>
+<label x="92.71" y="156.21" size="1.27" layer="95" xref="yes"/>
+<pinref part="U1" gate="G$1" pin="IO16"/>
+</segment>
+</net>
+<net name="SPI_MOSI" class="0">
+<segment>
+<wire x1="92.71" y1="153.67" x2="91.44" y2="153.67" width="0.1524" layer="91"/>
+<label x="92.71" y="153.67" size="1.27" layer="95" xref="yes"/>
+<pinref part="U1" gate="G$1" pin="IO17"/>
+</segment>
+</net>
+<net name="SPI_SCK" class="0">
+<segment>
+<wire x1="92.71" y1="151.13" x2="91.44" y2="151.13" width="0.1524" layer="91"/>
+<label x="92.71" y="151.13" size="1.27" layer="95" xref="yes"/>
+<pinref part="U1" gate="G$1" pin="IO18"/>
+</segment>
+</net>
+<net name="I2C_SCL" class="0">
+<segment>
+<wire x1="92.71" y1="143.51" x2="91.44" y2="143.51" width="0.1524" layer="91"/>
+<label x="92.71" y="143.51" size="1.27" layer="95" xref="yes"/>
+<pinref part="U1" gate="G$1" pin="IO22"/>
+</segment>
+</net>
+<net name="I2C_SDA" class="0">
+<segment>
+<wire x1="92.71" y1="140.97" x2="91.44" y2="140.97" width="0.1524" layer="91"/>
+<label x="92.71" y="140.97" size="1.27" layer="95" xref="yes"/>
+<pinref part="U1" gate="G$1" pin="IO23"/>
+</segment>
+</net>
+<net name="LED_CTRL" class="0">
+<segment>
+<pinref part="U1" gate="G$1" pin="IO19"/>
+<wire x1="92.71" y1="148.59" x2="91.44" y2="148.59" width="0.1524" layer="91"/>
+<label x="92.71" y="148.59" size="1.27" layer="95" xref="yes"/>
+</segment>
+</net>
+<net name="SPI_CS" class="0">
+<segment>
+<wire x1="92.71" y1="146.05" x2="91.44" y2="146.05" width="0.1524" layer="91"/>
+<label x="92.71" y="146.05" size="1.27" layer="95" xref="yes"/>
+<pinref part="U1" gate="G$1" pin="IO21"/>
+</segment>
+</net>
+<net name="STRAP_4" class="0">
+<segment>
+<wire x1="91.44" y1="168.91" x2="92.71" y2="168.91" width="0.1524" layer="91"/>
+<label x="92.71" y="168.91" size="1.27" layer="95" xref="yes"/>
+<pinref part="U1" gate="G$1" pin="IO5"/>
+</segment>
+</net>
+<net name="STRAP_0" class="0">
+<segment>
+<wire x1="132.08" y1="166.37" x2="133.35" y2="166.37" width="0.1524" layer="91"/>
+<label x="133.35" y="166.37" size="1.27" layer="95" xref="yes"/>
+</segment>
+</net>
+<net name="STRAP_1" class="0">
+<segment>
+<wire x1="91.44" y1="176.53" x2="92.71" y2="176.53" width="0.1524" layer="91"/>
+<label x="92.71" y="176.53" size="1.27" layer="95" xref="yes"/>
+<pinref part="U1" gate="G$1" pin="IO0"/>
+</segment>
+</net>
+<net name="STRAP_2" class="0">
+<segment>
+<wire x1="132.08" y1="162.56" x2="133.35" y2="162.56" width="0.1524" layer="91"/>
+<label x="133.35" y="162.56" size="1.27" layer="95" xref="yes"/>
+</segment>
+</net>
+<net name="STRAP_3" class="0">
+<segment>
+<wire x1="132.08" y1="157.48" x2="133.35" y2="157.48" width="0.1524" layer="91"/>
+<label x="133.35" y="157.48" size="1.27" layer="95" xref="yes"/>
+</segment>
+</net>

Commit message: deleted extra page
Parts:
- removed FD1, FD2: FIDUCIAL1X2, SparkFun-Aesthetics:FIDUCIAL1X2
- removed J4: FTSH-105-01-F-DV-K-TRJ, epoch:FTSH-105-01-F-DV-K-TRJ
- added D2: 1655, epoch:1655
Connections:
- new net N$6: D1.DOUT, D2.DIN
- new net SENSE_INT: U1.IO26, U2.INT1
- net +3V3: now also J2.SUPPLY_VOLTAGE, U2.VDD
- net GND: now also D1.VSS, D2.VSS, J2.SHIELD, J2.SUPPLY_VOLTAGE_GROUND, U2.GND
- net LED_CTRL: now also D1.DIN
- net SD_CLK: now also J2.CLOCK
- net SD_CMD: now also J2.COMMAND/RESPONSE
- net SD_D0: now also J2.DATA_LINE[BIT_0]
- net SD_D1: now also J2.DATA_LINE[BIT_1]
- net SD_D2: now also J2.DATA_LINE[BIT_2]
- net SD_D3: now also J2.CARD_DETECT/DATA_LINE[BIT_3]
- net SPI_CS: now also U2.NCS
- net SPI_MISO: now also U2.AD0/SDO
- net SPI_MOSI: now also U2.SDA/SDI
- net SPI_SCK: now also U2.SCL/SCLK
Other:
- note added: "0 ohm to mcu nrst"
- note added: "Add 10Ks for PUR?"
- note added: "Add 2-pin jst"
- note added: "Add diodes to switch input"
- note added: "Add led out pin"
- note added: "Insert AP1603WG-7 for 5v led"
- note added: "Wire usb"
- note removed: "Pullups"

Commit message: added rf components
Parts:
- removed U3: NEO-M8Q, epoch:NEO-M8Q
- removed U4: USBLC6-2P6, epoch:USBLC6-2P6
- added B1: 6.8MM_COIN_CELL, SparkFun-Batteries:ML414H_IV01E_BATTERY
- added C1, C2, C7, C9: 0.1uF, epoch:CAP_0603
- added C3, C4, C6: 1.0uF, SparkFun-Capacitors:1.0UF-0603-16V-10%
- added C5: 0.1uF, SparkFun-Capacitors:0.1UF-0603-25V-(+80/-20%)
- added C8: 22uF, epoch:CAP_0603
- added D3: 0.5A/40V/420mV, SparkFun-DiscreteSemi:DIODE-SCHOTTKY-PMEG4005EJ
- added D4: PRTR5V0U2F, SparkFun-IC-Power:PRTR5V0U2F
- added E1: ANT8010LL05R1516A, epoch:ANT8010LL05R1516A
- added J10: (no value), SparkFun-Connectors:JST_2MM_MALE
- added J4: Qwiic Right Angle, SparkFun-Connectors:I2C_STANDARDQWIIC
- added J6: (no value), SparkFun-Connectors:CONN_07NO_SILK
- added J8: (no value), SparkFun-Connectors:USB_C2-LAYER
- added J9: USB4105-GF-A, epoch:USB4105-GF-A
- added JP15: (no value), SparkFun-Connectors:CONN_041X04_NO_SILK
- added JP5: JUMPER-SMT_3_2-NC_TRACE_SILK, SparkFun-Jumpers:JUMPER-SMT_3_2-NC_TRACE_SILK
- added L1: 33nH/±5%/500mA, SparkFun-Coils:INDUCTOR-0603-33NH
- added R10, R9: 27, SparkFun-Resistors:27OHM-0603-1/10W-1%
- added R12, R13: 5.1k, SparkFun-Resistors:5.1KOHM5.1KOHM-0603-1/10W-1%
- added R15: 100k, SparkFun-Resistors:100KOHM-0603-1/10W-1%
- added R17: 10K, epoch:RES_0603
- added R2, R3, R4, R6: 33, SparkFun-Resistors:33OHM-0603-1/10W-1%
- added R5: 1k, SparkFun-Resistors:1KOHM-0603-1/10W-1%
- added R7, R8: 2.2k, SparkFun-Resistors:2.2KOHM-0603-1/10W-1%
- added S2: EG1213, epoch:EG1213
- added U10: USBLC6-2P6, epoch:USBLC6-2P6
- added U7: 3.3V, SparkFun-IC-Power:V_REG_AP2112K-3.3V
- added U8: U-BLOX_NEO-M9N, gps:U-BLOX_NEO-M9N
- added Y1: GPS_CHIP_ANTENNAW3011, SparkFun-GPS:GPS_CHIP_ANTENNAW3011
- J2: value 1140084168 -> FTSH-105-01-F-DV-K-TRJ; device epoch:1140084168 -> epoch:FTSH-105-01-F-DV-K-TRJ
- J3: value 105450-0101 -> 1140084168; device epoch:105450-0101 -> epoch:1140084168
- U1: value ESP32-WROOM-32D -> ICM-20948; device epoch:ESP32-WROOM-32D -> epoch:ICM-20948
- U2: value ICM-20948 -> ESP32-WROVER-B; device epoch:ICM-20948 -> epoch:ESP32-WROVER-B_(16MB)
Connections:
- removed net SENSE_INT: U1.IO26, U2.INT1
- removed net SPI_CS: U1.IO21, U2.NCS
- new net !RESET: JP15.3
- new net !SAFE: JP15.2
- new net 3.3V: C4.1, C5.2, D3.A, J4.2, J6.3, JP5.2, R15.2
- new net 5V: C6.1, D4.5, J6.2, J8.VBUS
- new net BACKUP: B1.+, C3.1, R5.1
- new net D+: D4.4, R9.1
- new net D-: D4.6, R10.1
- new net GPS_ANT1: Y1.SIGNAL
- new net IMU_INT: U1.INT1, U2.IO26/GPIO26
- new net INT: JP15.1
- new net N$1: D3.C, R5.2
- new net N$11: R9.2
- new net N$12: R10.2
- new net N$13: C9.1, S1.B'
- new net N$14: C9.2, S1.A'
- new net N$5: JP5.1, R8.2
- new net N$7: J8.CC2, R12.2
- new net N$8: JP5.3, R7.2
- new net N$9: J8.CC1, R13.2
- new net PPS: JP15.4
- new net RESET: S1.A, U2.EN
- new net RXI/MOSI: J6.5, R6.2
- new net RXLV: R6.1
- new net SCL/SCK: J4.4, J6.7, R4.2, R7.1
- new net SCL_LV: R4.1
- new net SDA/!CS: J4.3, J6.4, R2.2, R8.1
- new net SDA_LV: R2.1
- new net SHLD: J8.SHLD
- new net SPI_IMU_CS: R17.1, U1.NCS, U2.IO27/GPIO27
- new net STRAP_2: U2.IO2/GPIO2
- new net STRAP_3: U2.IO15/GPIO15
- new net TXLV: R3.1
- new net TXO/MISO: J6.6, R3.2
- new net USB_D+: D4.3, J8.D+
- new net USB_D-: D4.1, J8.D-
- net +3V3: now also C1.1, C2.1, C7.1, C8.1, J3.SUPPLY_VOLTAGE, R17.2, S1.B, U1.VDD, U2.3V3; no longer J2.SUPPLY_VOLTAGE, U1.3V3, U1.EN, U2.VDD
- net GND: now also B1.-, C1.2, C2.2, C3.2, C4.2, C5.1, C6.2, C7.2, C8.2, D4.2, J3.SHIELD, J3.SUPPLY_VOLTAGE_GROUND, J4.1, J6.1, J8.GND, R12.1, R13.1, R15.1, U2.EP, Y1.GND; no longer J2.SHIELD, J2.SUPPLY_VOLTAGE_GROUND
- net I2C_SCL: now also U2.IO35/GPIO35; no longer U1.IO22
- net I2C_SDA: now also U2.IO34/GPIO34; no longer U1.IO23
- net LED_CTRL: now also U2.IO33/GPIO33; no longer U1.IO19
- net RXD: now also U2.RXD0; no longer U1.RXD0
- net SD_CLK: now also J3.CLOCK; no longer J2.CLOCK, U1.IO14
- net SD_CMD: now also J3.COMMAND/RESPONSE; no longer J2.COMMAND/RESPONSE, U1.IO15
- net SD_D0: now also J3.DATA_LINE[BIT_0]; no longer J2.DATA_LINE[BIT_0], U1.IO2
- net SD_D1: now also J3.DATA_LINE[BIT_1]; no longer J2.DATA_LINE[BIT_1], U1.IO4
- net SD_D2: now also J3.DATA_LINE[BIT_2]; no longer J2.DATA_LINE[BIT_2], U1.IO12
- net SD_D3: now also J3.CARD_DETECT/DATA_LINE[BIT_3]; no longer J2.CARD_DETECT/DATA_LINE[BIT_3], U1.IO13
- net SPI_MISO: now also U1.AD0/SDO, U2.IO12/GPIO12; no longer U1.IO16, U2.AD0/SDO
- net SPI_MOSI: now also U1.SDA/SDI, U2.IO13/GPIO13; no longer U1.IO17, U2.SDA/SDI
- net SPI_SCK: now also U1.SCL/SCLK, U2.IO14/GPIO14; no longer U1.IO18, U2.SCL/SCLK
- net STRAP_1: now also U2.IO0/GPIO0; no longer U1.IO0
- net STRAP_4: now also U2.IO5/GPIO5; no longer U1.IO5
- net TXD: now also U2.TXD0; no longer U1.TXD0
Other:
- note added: "65 mil transmission line"
- note added: "7-bit unshifted I2C address: 0x42"
- note added: "Chip Antenna"
- note added: "Cut jumper to remove I2C pullups from bus"
- note added: "GPS"
- note added: "GPS: u-Blox NEO-M9N"
- note added: "Headers"
- note added: "Hot Start Battery"
- note added: "IMU"
- note added: "LEDs and Jumpers"
- note added: "Pullup Restors"
- note added: "SD Card"
- note added: "USB Connector - Power"
- note added: "VCC Range: 2.7V - 3.3V"

Commit message: finished schematic
Parts:
- removed B1: 6.8MM_COIN_CELL, SparkFun-Batteries:ML414H_IV01E_BATTERY
- removed E1: ANT8010LL05R1516A, epoch:ANT8010LL05R1516A
- removed J10: (no value), SparkFun-Connectors:JST_2MM_MALE
- removed J4: Qwiic Right Angle, SparkFun-Connectors:I2C_STANDARDQWIIC
- removed J6: (no value), SparkFun-Connectors:CONN_07NO_SILK
- removed J8: (no value), SparkFun-Connectors:USB_C2-LAYER
- removed J9: USB4105-GF-A, epoch:USB4105-GF-A
- removed JP15: (no value), SparkFun-Connectors:CONN_041X04_NO_SILK
- removed JP5: JUMPER-SMT_3_2-NC_TRACE_SILK, SparkFun-Jumpers:JUMPER-SMT_3_2-NC_TRACE_SILK
- removed L1: 33nH/±5%/500mA, SparkFun-Coils:INDUCTOR-0603-33NH
- removed U10: USBLC6-2P6, epoch:USBLC6-2P6
- removed U7: 3.3V, SparkFun-IC-Power:V_REG_AP2112K-3.3V
- removed U8: U-BLOX_NEO-M9N, gps:U-BLOX_NEO-M9N
- added BT1: ML414H-IV01E, SparkFun-Batteries:ML414H_IV01E_BATTERY
- added C10, C11, C12: 1uF, epoch:CAP_0603
- added D5: HSMD-C191, epoch:HSMD-C191
- added JP1: (no value), DC_LOAD_AU:PINHD-1X2
- added LOGO1: OSHW-LOGOMINI, SparkFun-Aesthetics:OSHW-LOGOMINI
- added R1: 0R, epoch:RES_0603
- added R11: 22R, epoch:RES_0603
- added R14: 0R DNI, epoch:RES_0603
- added R16: 5.1K, epoch:RES_0603
- added R18: 1.5K, epoch:RES_0603
- added U3: U-BLOX_NEO-M9N, gps:U-BLOX_NEO-M9N
- added U4: USBLC6-2P6, epoch:USBLC6-2P6
- C2: value 0.1uF -> 22uF
- C3, C4, C6: value 1.0uF -> 0.1uF; device SparkFun-Capacitors:1.0UF-0603-16V-10% -> epoch:CAP_0603
- C5: value 0.1uF -> 1uF; device SparkFun-Capacitors:0.1UF-0603-25V-(+80/-20%) -> epoch:CAP_0603
- C8: value 22uF -> 4.7uF
- C9: value 0.1uF -> 1uF
- D1: value 1655 -> 0.5A/40V/420mV; device epoch:1655 -> SparkFun-DiscreteSemi:DIODE-SCHOTTKY-PMEG4005EJ
- D2: value 1655 -> HSMN-C190; device epoch:1655 -> epoch:HSMN-C190
- D3: value 0.5A/40V/420mV -> BAT20JFILM; device SparkFun-DiscreteSemi:DIODE-SCHOTTKY-PMEG4005EJ -> SparkFun-DiscreteSemi:DIODE-SCHOTTKY-BAT20J
- D4: value PRTR5V0U2F -> HSMG-C190; device SparkFun-IC-Power:PRTR5V0U2F -> epoch:HSMG-C190
- J2: value FTSH-105-01-F-DV-K-TRJ -> USB4105-GF-A; device epoch:FTSH-105-01-F-DV-K-TRJ -> epoch:USB4105-GF-A
- J3: value 1140084168 -> (none); device epoch:1140084168 -> SparkFun-Connectors:JST_2MM_MALE
- R10: value 27 -> 1K; device SparkFun-Resistors:27OHM-0603-1/10W-1% -> epoch:RES_0603
- R12: value 5.1k -> 22R; device SparkFun-Resistors:5.1KOHM5.1KOHM-0603-1/10W-1% -> epoch:RES_0603
- R13: value 5.1k -> 0R DNI; device SparkFun-Resistors:5.1KOHM5.1KOHM-0603-1/10W-1% -> epoch:RES_0603
- R15: value 100k -> 5.1K; device SparkFun-Resistors:100KOHM-0603-1/10W-1% -> epoch:RES_0603
- R17: value 10K -> 1.5K
- R2: value 33 -> 100K DNI; device SparkFun-Resistors:33OHM-0603-1/10W-1% -> epoch:RES_0603
- R3: value 33 -> 10K; device SparkFun-Resistors:33OHM-0603-1/10W-1% -> epoch:RES_0603
- R4, R6: value 33 -> 0R DNI; device SparkFun-Resistors:33OHM-0603-1/10W-1% -> epoch:RES_0603
- R5: value 1k -> 0R DNI; device SparkFun-Resistors:1KOHM-0603-1/10W-1% -> epoch:RES_0603
- R7, R8: value 2.2k -> 0R DNI; device SparkFun-Resistors:2.2KOHM-0603-1/10W-1% -> epoch:RES_0603
- R9: value 27 -> 1.5K; device SparkFun-Resistors:27OHM-0603-1/10W-1% -> epoch:RES_0603
- U1: value ICM-20948 -> ESP32-WROVER-B; device epoch:ICM-20948 -> epoch:ESP32-WROVER-B_(16MB)
- U2: value ESP32-WROVER-B -> ICM-20948; device epoch:ESP32-WROVER-B_(16MB) -> epoch:ICM-20948
- U6: value TPS613221ADBVR -> 3.3V; device epoch:TPS613221ADBVR -> SparkFun-IC-Power:V_REG_AP2112K-3.3V
- Y1: value GPS_CHIP_ANTENNAW3011 -> W3011
Connections:
- removed net !RESET: JP15.3
- removed net !SAFE: JP15.2
- removed net 3.3V: C4.1, C5.2, D3.A, J4.2, J6.3, JP5.2, R15.2
- removed net 5V: C6.1, D4.5, J6.2, J8.VBUS
- removed net BACKUP: B1.+, C3.1, R5.1
- removed net D+: D4.4, R9.1
- removed net D-: D4.6, R10.1
- removed net GPS_ANT1: Y1.SIGNAL
- removed net INT: JP15.1
- removed net LED_CTRL: D1.DIN, U2.IO33/GPIO33
- removed net N$11: R9.2
- removed net N$12: R10.2
- removed net N$13: C9.1, S1.B'
- removed net N$14: C9.2, S1.A'
- removed net N$8: JP5.3, R7.2
- removed net N$9: J8.CC1, R13.2
- removed net RESET: S1.A, U2.EN
- removed net RXI/MOSI: J6.5, R6.2
- removed net RXLV: R6.1
- removed net SCL/SCK: J4.4, J6.7, R4.2, R7.1
- removed net SCL_LV: R4.1
- removed net SDA/!CS: J4.3, J6.4, R2.2, R8.1
- removed net SDA_LV: R2.1
- removed net SD_CLK: J3.CLOCK
- removed net SD_CMD: J3.COMMAND/RESPONSE
- removed net SD_D0: J3.DATA_LINE[BIT_0]
- removed net SD_D1: J3.DATA_LINE[BIT_1]
- removed net SD_D2: J3.DATA_LINE[BIT_2]
- removed net SD_D3: J3.CARD_DETECT/DATA_LINE[BIT_3]
- removed net SHLD: J8.SHLD
- removed net TXLV: R3.1
- removed net TXO/MISO: J6.6, R3.2
- removed net USB_D+: D4.3, J8.D+
- removed net USB_D-: D4.1, J8.D-
- new net ANTENNA: U3.RF_IN, Y1.SIGNAL
- new net BATTERY: C10.1, J3.+, S2.3, U5.VBAT
- new net BOARD_POWER: C11.1, D3.C, U6.EN, U6.IN
- new net BOOT: R13.1, U3.!SAFEBOOT!
- new net GPS_DN: R12.1, U4.I/O2_2
- new net GPS_DP: R11.1, U4.I/O1_2
- new net GPS_RESET: R14.1, U3.!RST
- new net HOTFIX_BATT: BT1.+, C5.1, R10.1, U3.V_BKCP
- new net MCU_RESET: C3.1, S1.B, U1.EN
- new net N$2: R11.2, U3.USB_D+
- new net N$3: R12.2, U3.USB_D-
- new net N$4: D2.A, R9.2
- new net STRAP_0: R1.2, R4.1
- new net USB_CC1: J2.CC1, R15.1
- new net USB_CC2: J2.CC2, R16.1
- new net USB_DN: J2.DN1, J2.DN2, U4.I/O2_1
- new net USB_DP: J2.DP1, J2.DP2, U4.I/O1_1
- new net VCC: C7.1, C8.1, C9.1, J2.VBUS, R17.1, U4.VBUS, U5.CE, U5.PROG, U5.VDD
- net +3V3: now also C12.1, C4.1, C6.1, D1.A, J1.2, R18.2, R3.2, U1.3V3, U2.VDD, U3.VCC, U3.VDD_USB, U6.OUT; no longer C7.1, C8.1, J3.SUPPLY_VOLTAGE, R17.2, S1.B, U1.VDD, U2.3V3
- net GND: now also BT1.-, C10.2, C11.2, C12.2, C5.2, C9.2, D2.C, D4.C, D5.C, J1.1, J2.GND, J3.-, JP1.2, R13.2, R14.2, R15.2, R16.2, R2.2, R4.2, R5.2, R6.2, R7.2, R8.2, S1.A, U1.EP, U3.GND, U4.GND, U5.VSS, U6.GND; no longer B1.-, C5.1, D1.VSS, D2.VSS, D4.2, J3.SHIELD, J3.SUPPLY_VOLTAGE_GROUND, J4.1, J6.1, J8.GND, R12.1, R13.1, R15.1, U2.EP
- net I2C_SCL: now also J1.3, U1.IO35/GPIO35, U3.SCL/SPI_CLK; no longer U2.IO35/GPIO35
- net I2C_SDA: now also J1.4, U1.IO34/GPIO34, U3.SDA/SPI_!CS!; no longer U2.IO34/GPIO34
- net IMU_INT: now also U1.IO26/GPIO26, U2.INT1; no longer U1.INT1, U2.IO26/GPIO26
- net N$1: now also D1.C, R10.2; no longer D3.C, R5.2
- net N$5: now also D5.A, R18.1; no longer JP5.1, R8.2
- net N$6: now also D4.A, R17.2; no longer D1.DOUT, D2.DIN
- net N$7: now also D3.A, S2.2; no longer J8.CC2, R12.2
- net PPS: now also R9.1, U3.TIMEPULSE; no longer JP15.4
- net RXD: now also U1.RXD0; no longer U2.RXD0
- net SPI_IMU_CS: now also R3.1, U1.IO27/GPIO27, U2.NCS; no longer R17.1, U1.NCS, U2.IO27/GPIO27
- net SPI_MISO: now also R1.1, R2.1, U1.IO12/GPIO12, U2.AD0/SDO; no longer U1.AD0/SDO, U2.IO12/GPIO12
- net SPI_MOSI: now also U1.IO13/GPIO13, U2.SDA/SDI; no longer U1.SDA/SDI, U2.IO13/GPIO13
- net SPI_SCK: now also U1.IO14/GPIO14, U2.SCL/SCLK; no longer U1.SCL/SCLK, U2.IO14/GPIO14
- net STRAP_1: now also JP1.1, R5.1, U1.IO0/GPIO0; no longer U2.IO0/GPIO0
- net STRAP_2: now also R6.1, U1.IO2/GPIO2; no longer U2.IO2/GPIO2
- net STRAP_3: now also R7.1, U1.IO15/GPIO15; no longer U2.IO15/GPIO15
- net STRAP_4: now also R8.1, U1.IO5/GPIO5; no longer U2.IO5/GPIO5
- net TXD: now also U1.TXD0; no longer U2.TXD0
Other:
- note added: "3.3V LDO"
- note added: "Charging Indicator"
- note added: "Debug Options"
- note added: "ESD Suppression"
- note added: "External I2C Connector"
- note added: "GPS Antenna"
- note added: "MCU Reset"
- note added: "On-board Battery and Charger"
- note added: "Power Indicator"
- note added: "Power Selection"
- note added: "Pullup/Pulldown"
- note added: "Pulse Per Second LED"
- note added: "USB"
- note removed: "0 ohm to mcu nrst"
- note removed: "65 mil transmission line"
- note removed: "7-bit unshifted I2C address: 0x42"
- note removed: "Add 10Ks for PUR?"
- note removed: "Add 2-pin jst"
- note removed: "Add diodes to switch input"
- note removed: "Add led out pin"
- note removed: "Chip Antenna"
- note removed: "Cut jumper to remove I2C pullups from bus"
- note removed: "GPS: u-Blox NEO-M9N"
- note removed: "Headers"
- note removed: "Hot Start Battery"
- note removed: "Insert AP1603WG-7 for 5v led"
- note removed: "LEDs and Jumpers"
- note removed: "Pullup Restors"
- note removed: "SD Card"
- note removed: "USB Connector - Power"
- note removed: "VCC Range: 2.7V - 3.3V"
- note removed: "Wire usb"
