File: boards/rev_A/epoch_revA.sch (EAGLE design)
At the start: 50 parts, among them J1 Qwiic Right Angle, J2 USB4105-GF-A, U1 ESP32-WROVER-B, U2 ICM-20948, U3 U-BLOX_NEO-M9N, U4 USBLC6-2P6, U5 MCP73811T-420I/OT, U6 3.3V, Y1 W3011

Commit message: working on layout
Parts:
- added C13, C14: 1uF, epoch:CAP_0603
- C10: value 1uF -> 4.7uF
- C5, C9: value 1uF -> 0.1uF
- C6: value 0.1uF -> 1uF
- C8: value 4.7uF -> 0.1uF
- U2: value ICM-20948 -> BMX160; device epoch:ICM-20948 -> epoch:BMX160
Connections:
- net N$2 renamed DP
- net N$3 renamed DN
- net +3V3: now also C14.1, C5.1, C7.1, C8.1, U2.VDDIO; no longer C12.1, C6.1
- net BATTERY: now also C12.1; no longer C10.1
- net BOARD_POWER: now also C13.1; no longer C11.1
- net GND: now also C13.2, C14.2, U2.GNDIO
- net HOTFIX_BATT: now also C6.1; no longer C5.1
- net SPI_IMU_CS: now also U2.CSB; no longer U2.NCS
- net SPI_MISO: now also U2.SDO; no longer U2.AD0/SDO
- net SPI_MOSI: now also U2.SDX; no longer U2.SDA/SDI
- net SPI_SCK: now also U2.SCX; no longer U2.SCL/SCLK
- net VCC: now also C10.1, C11.1; no longer C7.1, C8.1
Other:
- moved on the sheet: C11, C12, C4, C6, C7, C8
