File: boards/rev_A/epoch_revA.brd (EAGLE design)
At the start: 160 x 100 mm, 16 parts, among them J1 Qwiic Right Angle, J2 1140084168, J3 105450-0101, J4 FTSH-105-01-F-DV-K-TRJ, U1 ESP32-WROOM-32D, U2 ICM-20948, U3 NEO-M8Q, U4 USBLC6-2P6, U5 MCP73811T-420I/OT, U6 TPS613221ADBVR

Commit message: started defining board outline
Parts:
- added FD1, FD2: FIDUCIAL1X2, SparkFun-Aesthetics:FIDUCIAL-1X2
- moved C57 168.6 mm to (61.2, -4.57)
- moved R37 168.6 mm to (65.0, -4.57)
- moved R39 168.6 mm to (54.9, -8.38)
- moved R40 168.6 mm to (58.7, -8.38)
- moved U4 121.7 mm to (23.9, -23.4)
- moved D1 121.7 mm to (56.9, 2.03)
- moved J1 121.7 mm to (79.8, 2.03)
- moved J2 121.7 mm to (68.3, 3.30)
- moved J4 121.7 mm to (41.7, -19.6)
- moved S1 121.7 mm to (32.8, -8.13)
- moved U2 121.7 mm to (95.0, 8.38)
- moved U5 121.7 mm to (18.8, -22.1)
- moved U6 121.7 mm to (12.4, -22.1)
- moved J3 69.4 mm to (-9.14, 23.4), turned to 270 degrees
- moved U3 61.7 mm to (23.6, 11.7), turned to 90 degrees
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Connections:
- removed net 3V3: U1.2
- new net N$2: R37.2, R39.2, R40.2
- new net SD_CLK: U1.13
- new net SD_CMD: U1.23
- new net SD_D0: U1.24
- new net SD_D1: U1.26
- new net SD_D2: U1.14
- new net SD_D3: U1.16
- net +3V3: now also U1.2, U1.3; no longer R37.2, R39.2, R40.2
- net GND: now also U1.THERM1, U1.THERM2, U1.THERM3, U1.THERM4, U1.THERM5, U1.THERM6, U1.THERM7, U1.THERM8, U1.THERM9
Other:
- board size 160 x 100 mm -> 38.1 x 50.8 mm

Commit message: working on pin connections
Parts:
- removed C57: 10uF, Resistor_Capacitor:CAP_0402
- removed R37, R39, R40: 10K, Resistor_Capacitor:RES_0402
Connections:
- removed net FPGA_CS: R37.1
- removed net HOLD: R40.1
- removed net N$2: R37.2, R39.2, R40.2
- removed net WP: R39.1
- new net I2C_SCL: U1.36
- new net I2C_SDA: U1.37
- new net LED_CTRL: U1.31
- new net RXD: U1.34
- new net SPI_CS: U1.33
- new net SPI_MISO: U1.27
- new net SPI_MOSI: U1.28
- new net SPI_SCK: U1.30
- new net STRAP_1: U1.25
- new net STRAP_4: U1.29
- new net TXD: U1.35
- net GND: no longer C57.2
- net VCC: no longer C57.1
Changed lines of the file:
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@@
 <attribute name="VALUE" x="10.446" y="-24.698" size="0.8128" layer="27"/>
-</element>
-<element name="R39" library="Resistor_Capacitor" library_urn="urn:adsk.eagle:library:11396451" package="RES_0402" package3d_urn="urn:adsk.eagle:package:10872901/3" value="10K" x="54.864" y="-8.382" smashed="yes">
-<attribute name="CREATED_BY" value="PCBLayout.com" x="39.624" y="8.128" size="1.778" layer="27" display="off"/>
-<attribute name="DIGIKEY_PART_NUMBER" value="" x="39.624" y="8.128" size="1.778" layer="27" display="off"/>
-<attribute name="MANUFACTURER" value="Yageo" x="39.624" y="8.128" size="1.778" layer="27" display="off"/>
-<attribute name="MPN" value="AC0402FR-1310KL" x="39.624" y="8.128" size="1.778" layer="27" display="off"/>
-<attribute name="NAME" x="53.594" y="-7.874" size="0.5" layer="25" ratio="10"/>
-<attribute name="PACKAGE" value="SMD 0402" x="39.624" y="8.128" size="1.778" layer="27" display="off"/>
-<attribute name="VALUE" x="53.594" y="-9.398" size="0.5" layer="27" ratio="10"/>
-</element>
-<element name="R40" library="Resistor_Capacitor" library_urn="urn:adsk.eagle:library:11396451" package="RES_0402" package3d_urn="urn:adsk.eagle:package:10872901/3" value="10K" x="58.674" y="-8.382" smashed="yes">
-<attribute name="CREATED_BY" value="PCBLayout.com" x="39.624" y="4.318" size="1.778" layer="27" display="off"/>
-<attribute name="DIGIKEY_PART_NUMBER" value="" x="39.624" y="4.318" size="1.778" layer="27" display="off"/>
-<attribute name="MANUFACTURER" value="Yageo" x="39.624" y="4.318" size="1.778" layer="27" display="off"/>
-<attribute name="MPN" value="AC0402FR-1310KL" x="39.624" y="4.318" size="1.778" layer="27" display="off"/>
-<attribute name="NAME" x="57.404" y="-7.874" size="0.5" layer="25" ratio="10"/>
-<attribute name="PACKAGE" value="SMD 0402" x="39.624" y="4.318" size="1.778" layer="27" display="off"/>
-<attribute name="VALUE" x="57.404" y="-9.398" size="0.5" layer="27" ratio="10"/>
-</element>
-<element name="R37" library="Resistor_Capacitor" library_urn="urn:adsk.eagle:library:11396451" package="RES_0402" package3d_urn="urn:adsk.eagle:package:10872901/3" value="10K" x="65.024" y="-4.572" smashed="yes">
-<attribute name="CREATED_BY" value="PCBLayout.com" x="39.624" y="0.508" size="1.778" layer="27" display="off"/>
-<attribute name="DIGIKEY_PART_NUMBER" value="" x="39.624" y="0.508" size="1.778" layer="27" display="off"/>
-<attribute name="MANUFACTURER" value="Yageo" x="39.624" y="0.508" size="1.778" layer="27" display="off"/>
-<attribute name="MPN" value="AC0402FR-1310KL" x="39.624" y="0.508" size="1.778" layer="27" display="off"/>
-<attribute name="NAME" x="63.754" y="-4.064" size="0.5" layer="25" ratio="10"/>
-<attribute name="PACKAGE" value="SMD 0402" x="39.624" y="0.508" size="1.778" layer="27" display="off"/>
-<attribute name="VALUE" x="63.754" y="-5.588" size="0.5" layer="27" ratio="10"/>
-</element>
-<element name="C57" library="Resistor_Capacitor" library_urn="urn:adsk.eagle:library:11396451" package="CAP_0402" package3d_urn="urn:adsk.eagle:package:10872910/2" value="10uF" x="61.214" y="-4.572" smashed="yes">
-<attribute name="CREATED_BY" value="PCBLayout.com" x="39.624" y="-3.302" size="1.778" layer="27" display="off"/>
-<attribute name="DIGIKEY_PART_NUMBER" value="" x="39.624" y="-3.302" size="1.778" layer="27" display="off"/>
-<attribute name="MANUFACTURER" value="Murata" x="39.624" y="-3.302" size="1.778" layer="27" display="off"/>
-<attribute name="MPN" value="GRM155C80G106ME44D" x="39.624" y="-3.302" size="1.778" layer="27" display="off"/>
-<attribute name="NAME" x="60.044" y="-3.972" size="0.5" layer="25" ratio="10"/>
-<attribute name="PACKAGE" value="SMD 0402" x="39.624" y="-3.302" size="1.778" layer="27" display="off"/>
-<attribute name="VALUE" x="60.124" y="-5.602" size="0.5" layer="27" ratio="10"/>
 </element>
 <element name="FD1" library="SparkFun-Aesthetics" library_urn="urn:adsk.eagle:library:507" package="FIDUCIAL-1X2" package3d_urn="urn:adsk.eagle:package:37108/1" value="FIDUCIAL1X2" x="52.832" y="-10.668" smashed="yes"/>
@@
 <contactref element="U4" pad="2"/>
 <contactref element="U6" pad="2"/>
-<contactref element="C57" pad="2"/>
 <contactref element="U1" pad="1"/>
 <contactref element="U1" pad="15"/>
@@
 <contactref element="U1" pad="THERM8"/>
 <contactref element="U1" pad="THERM9"/>
-<wire x1="61.689" y1="-4.572" x2="96.541" y2="9.382" width="0" layer="19" extent="1-1"/>
-<wire x1="30.622" y1="5.684" x2="61.689" y2="-4.572" width="0" layer="19" extent="1-1"/>
+<wire x1="30.622" y1="5.684" x2="96.541" y2="9.382" width="0" layer="19" extent="1-1"/>
 <wire x1="28.422" y1="5.684" x2="30.622" y2="5.684" width="0" layer="19" extent="1-1"/>
 <wire x1="30.622" y1="17.684" x2="30.622" y2="5.684" width="0" layer="19" extent="1-1"/>
@@
 <signal name="VCC">
 <contactref element="U3" pad="23"/>
-<contactref element="C57" pad="1"/>
-<wire x1="17.722" y1="17.684" x2="60.739" y2="-4.572" width="0" layer="19" extent="1-1"/>
 </signal>
 <signal name="VDD_USB">
@@
 <contactref element="U6" pad="4"/>
 </signal>
-<signal name="FPGA_CS">
-<contactref element="R37" pad="1"/>
-</signal>
-<signal name="WP">
-<contactref element="R39" pad="1"/>
-</signal>
-<signal name="HOLD">
-<contactref element="R40" pad="1"/>
-</signal>
 <signal name="N$1">
-</signal>
-<signal name="N$2">
-<contactref element="R40" pad="2"/>
-<contactref element="R39" pad="2"/>
-<contactref element="R37" pad="2"/>
-<wire x1="59.134" y1="-8.382" x2="65.484" y2="-4.572" width="0" layer="19" extent="1-1"/>
-<wire x1="55.324" y1="-8.382" x2="59.134" y2="-8.382" width="0" layer="19" extent="1-1"/>
 </signal>
 <signal name="+3V3">
@@
 <contactref element="U1" pad="26"/>
 </signal>
+<signal name="TXD">
+<contactref element="U1" pad="35"/>
+</signal>
+<signal name="RXD">
+<contactref element="U1" pad="34"/>
+</signal>
+<signal name="SPI_MISO">
+<contactref element="U1" pad="27"/>
+</signal>
+<signal name="SPI_MOSI">
+<contactref element="U1" pad="28"/>
+</signal>
+<signal name="SPI_SCK">
+<contactref element="U1" pad="30"/>
+</signal>
+<signal name="I2C_SCL">
+<contactref element="U1" pad="36"/>
+</signal>
+<signal name="I2C_SDA">
+<contactref element="U1" pad="37"/>
+</signal>
+<signal name="LED_CTRL">
+<contactref element="U1" pad="31"/>
+</signal>
+<signal name="SPI_CS">
+<contactref element="U1" pad="33"/>
+</signal>
+<signal name="STRAP_4">
+<contactref element="U1" pad="29"/>
+</signal>
+<signal name="STRAP_1">
+<contactref element="U1" pad="25"/>
+</signal>
+<signal name="STRAP_3">
+</signal>
 </signals>

Commit message: deleted extra page
Parts:
- removed FD1, FD2: FIDUCIAL1X2, SparkFun-Aesthetics:FIDUCIAL-1X2
- removed J4: FTSH-105-01-F-DV-K-TRJ, epoch:SAMTEC-FTSH-105-01-X-DV
- added D2: 1655, epoch:LED_1655
- moved U2 108.7 mm to (3.30, -50.0)
- moved U1 82.8 mm to (19.1, 37.6)
- moved J2 74.5 mm to (7.62, -39.9)
- moved J3 70.6 mm to (-9.65, -47.2), turned to 0 degrees
- moved U4 38.6 mm to (-2.29, -51.8)
Connections:
- removed net SUPPLY_VOLTAGE: J2.4
- removed net SUPPLY_VOLTAGE_GROUND: J2.6
- new net N$6: D1.4, D2.2
- new net SENSE_INT: U1.11, U2.12
- net +3V3: now also J2.4, U2.13
- net GND: now also D1.1, D2.1, J2.6, J2.S1, J2.S2, J2.S3, J2.S4
- net LED_CTRL: now also D1.2
- net SD_CLK: now also J2.5
- net SD_CMD: now also J2.3
- net SD_D0: now also J2.7
- net SD_D1: now also J2.8
- net SD_D2: now also J2.1
- net SD_D3: now also J2.2
- net SPI_CS: now also U2.22
- net SPI_MISO: now also U2.9
- net SPI_MOSI: now also U2.24
- net SPI_SCK: now also U2.23
- net VDD: now also D2.3; no longer U2.13
- net VSS: no longer D1.1

Commit message: added rf components
Parts:
- removed U3: NEO-M8Q, epoch:XCVR_NEO-M8Q
- removed U4: USBLC6-2P6, epoch:SOT50P160X60-6N
- added B1: 6.8MM_COIN_CELL, SparkFun-Batteries:ML414H_IV01E
- added C1, C2, C7, C9: 0.1uF, epoch:0603
- added C3, C4, C6: 1.0uF, SparkFun-Capacitors:0603
- added C5: 0.1uF, SparkFun-Capacitors:0603
- added C8: 22uF, epoch:0603
- added D3: 0.5A/40V/420mV, SparkFun-DiscreteSemi:SOD-323
- added D4: PRTR5V0U2F, SparkFun-IC-Power:SOT886
- added E1: ANT8010LL05R1516A, epoch:ANT8010LL05R1516A
- added J10: (no value), SparkFun-Connectors:JST-2-SMD
- added J4: Qwiic Right Angle, SparkFun-Connectors:JST04_1MM_RA
- added J6: (no value), SparkFun-Connectors:1X07_NO_SILK
- added J8: (no value), SparkFun-Connectors:USB-C-16P
- added J9: USB4105-GF-A, epoch:GCT_USB4105-GF-A
- added JP15: (no value), SparkFun-Connectors:1X04_NO_SILK
- added JP5: JUMPER-SMT_3_2-NC_TRACE_SILK, SparkFun-Jumpers:SMT-JUMPER_3_2-NC_TRACE_SILK
- added L1: 33nH/±5%/500mA, SparkFun-Coils:0603
- added R10, R9: 27, SparkFun-Resistors:0603
- added R12, R13: 5.1k, SparkFun-Resistors:0603
- added R15: 100k, SparkFun-Resistors:0603
- added R17: 10K, epoch:0603
- added R2, R3, R4, R6: 33, SparkFun-Resistors:0603
- added R5: 1k, SparkFun-Resistors:0603
- added R7, R8: 2.2k, SparkFun-Resistors:0603
- added S2: EG1213, epoch:SW_EG1213
- added U10: USBLC6-2P6, epoch:SOT50P160X60-6N
- added U7: 3.3V, SparkFun-IC-Power:SOT23-5
- added U8: U-BLOX_NEO-M9N, gps:NEO-M9N
- added Y1: GPS_CHIP_ANTENNAW3011, SparkFun-GPS:W3011
- J2: value 1140084168 -> FTSH-105-01-F-DV-K-TRJ; device epoch:AMPHENOL_1140084168 -> epoch:SAMTEC-FTSH-105-01-X-DV
- J3: value 105450-0101 -> 1140084168; device epoch:MOLEX_105450-0101 -> epoch:AMPHENOL_1140084168
- U1: value ESP32-WROOM-32D -> ICM-20948; device epoch:MODULE_ESP32-WROOM-32D -> epoch:QFN40P300X300X105-24N
- U2: value ICM-20948 -> ESP32-WROVER-B; device epoch:QFN40P300X300X105-24N -> epoch:XCVR_ESP32-WROVER-B_(16MB)
- moved S1 322.3 mm to (-122.4, -290.6)
- moved J2 293.5 mm to (-117.6, -305.3)
- moved U1 256.4 mm to (-77.0, -200.2)
- moved J3 192.4 mm to (-72.4, -229.1)
- moved U2 86.1 mm to (19.6, 34.5)
Connections:
- removed net SENSE_INT: U1.11, U2.12
- removed net SPI_CS: U1.33, U2.22
- removed net VCC: U3.23
- removed net VDD_USB: U3.7
- removed net V_BCKP: U3.22
- new net !RESET: JP15.3
- new net !SAFE: JP15.2
- new net 3.3V: C4.1, C5.2, D3.A, J4.2, J6.3, JP5.2, R15.2
- new net 5V: C6.1, D4.5, J6.2, J8.VBUS1, J8.VBUS2
- new net BACKUP: B1.+, C3.1, R5.1
- new net D+: D4.4, R9.1
- new net D-: D4.6, R10.1
- new net GPS_ANT1: Y1.1
- new net IMU_INT: U1.12, U2.11
- new net INT: JP15.1
- new net N$1: D3.C, R5.2
- new net N$11: R9.2
- new net N$12: R10.2
- new net N$13: C9.1, S1.B'
- new net N$14: C9.2, S1.A'
- new net N$5: JP5.1, R8.2
- new net N$7: J8.B5, R12.2
- new net N$8: JP5.3, R7.2
- new net N$9: J8.A5, R13.2
- new net PPS: JP15.4
- new net RESET: S1.A, U2.3
- new net RXI/MOSI: J6.5, R6.2
- new net RXLV: R6.1
- new net SCL/SCK: J4.4, J6.7, R4.2, R7.1
- new net SCL_LV: R4.1
- new net SDA/!CS: J4.3, J6.4, R2.2, R8.1
- new net SDA_LV: R2.1
- new net SHLD: J8.SHLD1, J8.SHLD2, J8.SHLD3, J8.SHLD4, J8.SHLD5, J8.SHLD6, J8.SHLD7, J8.SHLD8
- new net SPI_IMU_CS: R17.1, U1.22, U2.12
- new net STRAP_2: U2.24
- new net STRAP_3: U2.23
- new net TXLV: R3.1
- new net TXO/MISO: J6.6, R3.2
- new net USB_D+: D4.3, J8.A6, J8.B6
- new net USB_D-: D4.1, J8.A7, J8.B7
- net +3V3: now also C1.1, C2.1, C7.1, C8.1, J3.4, R17.2, S1.B, U1.13, U2.2; no longer J2.4, U1.2, U1.3, U2.13
- net GND: now also B1.-, C1.2, C2.2, C3.2, C4.2, C5.1, C6.2, C7.2, C8.2, D4.2, E1.SOLDER, J3.6, J3.S1, J3.S2, J3.S3, J3.S4, J4.1, J6.1, J8.GND, J8.GND2, J9.A1/B12, J9.B1/A12, J9.G1, J9.G2, J9.G3, J9.G4, R12.1, R13.1, R15.1, U1.18, U10.2, U2.1, U2.15, U2.38, U2.39, Y1.2, Y1.3; no longer J2.6, J2.S1, J2.S2, J2.S3, J2.S4, U1.1, U1.15, U1.38, U1.39, U1.THERM1, U1.THERM2, U1.THERM3, U1.THERM4, U1.THERM5, U1.THERM6, U1.THERM7, U1.THERM8, U1.THERM9, U2.18, U3.10, U3.12, U3.13, U3.24, U4.2
- net I2C_SCL: now also U2.7; no longer U1.36
- net I2C_SDA: now also U2.6; no longer U1.37
- net LED_CTRL: now also U2.9; no longer U1.31
- net RXD: now also U2.34; no longer U1.34
- net SD_CLK: now also J3.5; no longer J2.5, U1.13
- net SD_CMD: now also J3.3; no longer J2.3, U1.23
- net SD_D0: now also J3.7; no longer J2.7, U1.24
- net SD_D1: now also J3.8; no longer J2.8, U1.26
- net SD_D2: now also J3.1; no longer J2.1, U1.14
- net SD_D3: now also J3.2; no longer J2.2, U1.16
- net SPI_MISO: now also U1.9, U2.14; no longer U1.27, U2.9
- net SPI_MOSI: now also U1.24, U2.16; no longer U1.28, U2.24
- net SPI_SCK: now also U1.23, U2.13; no longer U1.30, U2.23
- net STRAP_1: now also U2.25; no longer U1.25
- net STRAP_4: now also U2.29; no longer U1.29
- net TXD: now also U2.35; no longer U1.35
- net VBUS: now also J9.A4/B9, J9.B4/A9, U10.5; no longer U4.5
- net VDDIO: now also U1.8; no longer U2.8

Commit message: finished schematic
Parts:
- removed B1: 6.8MM_COIN_CELL, SparkFun-Batteries:ML414H_IV01E
- removed E1: ANT8010LL05R1516A, epoch:ANT8010LL05R1516A
- removed J10: (no value), SparkFun-Connectors:JST-2-SMD
- removed J4: Qwiic Right Angle, SparkFun-Connectors:JST04_1MM_RA
- removed J6: (no value), SparkFun-Connectors:1X07_NO_SILK
- removed J8: (no value), SparkFun-Connectors:USB-C-16P
- removed J9: USB4105-GF-A, epoch:GCT_USB4105-GF-A
- removed JP15: (no value), SparkFun-Connectors:1X04_NO_SILK
- removed JP5: JUMPER-SMT_3_2-NC_TRACE_SILK, SparkFun-Jumpers:SMT-JUMPER_3_2-NC_TRACE_SILK
- removed L1: 33nH/±5%/500mA, SparkFun-Coils:0603
- removed U10: USBLC6-2P6, epoch:SOT50P160X60-6N
- removed U7: 3.3V, SparkFun-IC-Power:SOT23-5
- removed U8: U-BLOX_NEO-M9N, gps:NEO-M9N
- added BT1: ML414H-IV01E, SparkFun-Batteries:ML414H_IV01E
- added C10, C11, C12: 1uF, epoch:0603
- added D5: HSMD-C191, epoch:LEDM1608X80
- added JP1: (no value), DC_LOAD_AU:1X02
- added LOGO1: OSHW-LOGOMINI, SparkFun-Aesthetics:OSHW-LOGO-MINI
- added R1: 0R, epoch:0603
- added R11: 22R, epoch:0603
- added R14: 0R DNI, epoch:0603
- added R16: 5.1K, epoch:0603
- added R18: 1.5K, epoch:0603
- added U3: U-BLOX_NEO-M9N, gps:NEO-M9N
- added U4: USBLC6-2P6, epoch:SOT50P160X60-6N
- C2: value 0.1uF -> 22uF
- C3, C4, C6: value 1.0uF -> 0.1uF; device SparkFun-Capacitors:0603 -> epoch:0603
- C5: value 0.1uF -> 1uF; device SparkFun-Capacitors:0603 -> epoch:0603
- C8: value 22uF -> 4.7uF
- C9: value 0.1uF -> 1uF
- D1: value 1655 -> 0.5A/40V/420mV; device epoch:LED_1655 -> SparkFun-DiscreteSemi:SOD-323
- D2: value 1655 -> HSMN-C190; device epoch:LED_1655 -> epoch:LEDM1608X80
- D3: value 0.5A/40V/420mV -> BAT20JFILM
- D4: value PRTR5V0U2F -> HSMG-C190; device SparkFun-IC-Power:SOT886 -> epoch:LEDM1608X80
- J2: value FTSH-105-01-F-DV-K-TRJ -> USB4105-GF-A; device epoch:SAMTEC-FTSH-105-01-X-DV -> epoch:GCT_USB4105-GF-A
- J3: value 1140084168 -> (none); device epoch:AMPHENOL_1140084168 -> SparkFun-Connectors:JST-2-SMD
- R10: value 27 -> 1K; device SparkFun-Resistors:0603 -> epoch:0603
- R12: value 5.1k -> 22R; device SparkFun-Resistors:0603 -> epoch:0603
- R13: value 5.1k -> 0R DNI; device SparkFun-Resistors:0603 -> epoch:0603
- R15: value 100k -> 5.1K; device SparkFun-Resistors:0603 -> epoch:0603
- R17: value 10K -> 1.5K
- R2: value 33 -> 100K DNI; device SparkFun-Resistors:0603 -> epoch:0603
- R3: value 33 -> 10K; device SparkFun-Resistors:0603 -> epoch:0603
- R4, R6: value 33 -> 0R DNI; device SparkFun-Resistors:0603 -> epoch:0603
- R5: value 1k -> 0R DNI; device SparkFun-Resistors:0603 -> epoch:0603
- R7, R8: value 2.2k -> 0R DNI; device SparkFun-Resistors:0603 -> epoch:0603
- R9: value 27 -> 1.5K; device SparkFun-Resistors:0603 -> epoch:0603
- U1: value ICM-20948 -> ESP32-WROVER-B; device epoch:QFN40P300X300X105-24N -> epoch:XCVR_ESP32-WROVER-B_(16MB)
- U2: value ESP32-WROVER-B -> ICM-20948; device epoch:XCVR_ESP32-WROVER-B_(16MB) -> epoch:QFN40P300X300X105-24N
- U6: value TPS613221ADBVR -> 3.3V; device epoch:SOT95P280X145-5N -> SparkFun-IC-Power:SOT23-5
- Y1: value GPS_CHIP_ANTENNAW3011 -> W3011
- moved S1 380.6 mm to (95.8, 21.3)
- moved J2 340.2 mm to (2.54, 13.0), turned to 270 degrees
- moved C2 313.9 mm to (91.9, 26.9)
- moved C1 302.2 mm to (91.9, 43.2)
- moved S2 298.8 mm to (35.8, 37.6), turned to 90 degrees
- moved C8 273.6 mm to (-54.9, -20.8)
- moved C7 261.1 mm to (-54.9, -17.5)
- moved C9 255.0 mm to (-54.9, -52.6)
- moved U1 253.6 mm to (19.1, 34.5)
- moved C3 245.7 mm to (91.9, 14.5)
- moved J3 244.8 mm to (-32.5, 12.4)
- moved C4 187.8 mm to (117.1, 23.9)
- moved R13 172.5 mm to (56.9, 42.7)
- moved R12 160.0 mm to (-54.9, 36.1)
- moved R15 158.9 mm to (-54.9, 32.8)
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Connections:
- removed net !RESET: JP15.3
- removed net !SAFE: JP15.2
- removed net 1: J1.1
- removed net 2: J1.2
- removed net 3.3V: C4.1, C5.2, D3.A, J4.2, J6.3, JP5.2, R15.2
- removed net 5V: C6.1, D4.5, J6.2, J8.VBUS1, J8.VBUS2
- removed net BACKUP: B1.+, C3.1, R5.1
- removed net D+: D4.4, R9.1
- removed net D-: D4.6, R10.1
- removed net GPS_ANT1: Y1.1
- removed net INT: JP15.1
- removed net LED_CTRL: D1.2, U2.9
- removed net N$11: R9.2
- removed net N$12: R10.2
- removed net N$13: C9.1, S1.B'
- removed net N$14: C9.2, S1.A'
- removed net N$8: JP5.3, R7.2
- removed net N$9: J8.A5, R13.2
- removed net RESET: S1.A, U2.3
- removed net RXI/MOSI: J6.5, R6.2
- removed net RXLV: R6.1
- removed net SCL/SCK: J4.4, J6.7, R4.2, R7.1
- removed net SCL_LV: R4.1
- removed net SDA/!CS: J4.3, J6.4, R2.2, R8.1
- removed net SDA_LV: R2.1
- removed net SD_CLK: J3.5
- removed net SD_CMD: J3.3
- removed net SD_D0: J3.7
- removed net SD_D1: J3.8
- removed net SD_D2: J3.1
- removed net SD_D3: J3.2
- removed net SHLD: J8.SHLD1, J8.SHLD2, J8.SHLD3, J8.SHLD4, J8.SHLD5, J8.SHLD6, J8.SHLD7, J8.SHLD8
- removed net TXLV: R3.1
- removed net TXO/MISO: J6.6, R3.2
- removed net USB_D+: D4.3, J8.A6, J8.B6
- removed net USB_D-: D4.1, J8.A7, J8.B7
- removed net VBUS: J9.A4/B9, J9.B4/A9, U10.5
- removed net VDD: D1.3, D2.3, U5.4
- removed net VOUT: U6.4
- removed net VSS: U5.2
- new net ANTENNA: U3.11, Y1.1
- new net BATTERY: C10.1, J3.2, S2.3, U5.3
- new net BOARD_POWER: C11.1, D3.C, U6.1, U6.3
- new net BOOT: R13.1, U3.1
- new net GPS_DN: R12.1, U4.4
- new net GPS_DP: R11.1, U4.6
- new net GPS_RESET: R14.1, U3.8
- new net HOTFIX_BATT: BT1.+, C5.1, R10.1, U3.22
- new net MCU_RESET: C3.1, S1.B, U1.3
- new net N$2: R11.2, U3.6
- new net N$3: R12.2, U3.5
- new net N$4: D2.A, R9.2
- new net STRAP_0: R1.2, R4.1
- new net USB_CC1: J2.A5, R15.1
- new net USB_CC2: J2.B5, R16.1
- new net USB_DN: J2.A7, J2.B7, U4.3
- new net USB_DP: J2.A6, J2.B6, U4.1
- new net VCC: C7.1, C8.1, C9.1, J2.A4/B9, J2.B4/A9, R17.1, U4.5, U5.1, U5.4, U5.5
- net +3V3: now also C12.1, C4.1, C6.1, D1.A, J1.2, R18.2, R3.2, U1.2, U2.13, U3.23, U3.7, U6.5; no longer C7.1, C8.1, J3.4, R17.2, S1.B, U1.13, U2.2
- net GND: now also BT1.-, C10.2, C11.2, C12.2, C5.2, C9.2, D2.C, D4.C, D5.C, J1.1, J2.A1/B12, J2.B1/A12, J2.G1, J2.G2, J2.G3, J2.G4, J3.1, JP1.2, R13.2, R14.2, R15.2, R16.2, R2.2, R4.2, R5.2, R6.2, R7.2, R8.2, S1.A, U1.1, U1.15, U1.38, U1.39, U2.18, U3.10, U3.12, U3.13, U3.24, U4.2, U5.2; no longer B1.-, C5.1, D1.1, D2.1, D4.2, E1.SOLDER, J3.6, J3.S1, J3.S2, J3.S3, J3.S4, J4.1, J6.1, J8.GND, J8.GND2, J9.A1/B12, J9.B1/A12, J9.G1, J9.G2, J9.G3, J9.G4, R12.1, R13.1, R15.1, U1.18, U10.2, U2.1, U2.15, U2.38, U2.39
- net I2C_SCL: now also J1.3, U1.7, U3.19; no longer U2.7
- net I2C_SDA: now also J1.4, U1.6, U3.18; no longer U2.6
- net IMU_INT: now also U1.11, U2.12; no longer U1.12, U2.11
- net N$1: now also D1.C, R10.2; no longer D3.C, R5.2
- net N$5: now also D5.A, R18.1; no longer JP5.1, R8.2
- net N$6: now also D4.A, R17.2; no longer D1.4, D2.2
- net N$7: now also D3.A, S2.2; no longer J8.B5, R12.2
- net PPS: now also R9.1, U3.3; no longer JP15.4
- net RXD: now also U1.34; no longer U2.34
- net SPI_IMU_CS: now also R3.1, U1.12, U2.22; no longer R17.1, U1.22, U2.12
- net SPI_MISO: now also R1.1, R2.1, U1.14, U2.9; no longer U1.9, U2.14
- net SPI_MOSI: now also U1.16, U2.24; no longer U1.24, U2.16
- net SPI_SCK: now also U1.13, U2.23; no longer U1.23, U2.13
- net STRAP_1: now also JP1.1, R5.1, U1.25; no longer U2.25
- net STRAP_2: now also R6.1, U1.24; no longer U2.24
- net STRAP_3: now also R7.1, U1.23; no longer U2.23
- net STRAP_4: now also R8.1, U1.29; no longer U2.29
- net TXD: now also U1.35; no longer U2.35
- net VDDIO: now also U2.8; no longer U1.8

Commit message: working on layout
Parts:
- added C13, C14: 1uF, epoch:0603
- C10: value 1uF -> 4.7uF
- C5, C9: value 1uF -> 0.1uF
- C6: value 0.1uF -> 1uF
- C8: value 4.7uF -> 0.1uF
- U2: value ICM-20948 -> BMX160; device epoch:QFN40P300X300X105-24N -> epoch:PQFN50P250X300X100-14N
- moved C2 120.7 mm to (-27.9, 12.7)
- moved C4 114.5 mm to (3.05, 34.0), turned to 270 degrees
- moved U2 112.3 mm to (5.84, 34.3), turned to 270 degrees
- moved R1 106.8 mm to (-20.3, 15.2)
- moved R2 106.8 mm to (-20.3, 11.9)
- moved R3 106.8 mm to (-20.3, 28.4)
- moved R6 106.8 mm to (-20.3, 25.1)
- moved R7 106.8 mm to (-20.3, 21.8)
- moved R8 106.8 mm to (-20.3, 18.5)
- moved C10 100.4 mm to (11.4, 19.6), turned to 270 degrees
- moved C9 96.9 mm to (9.91, 19.6), turned to 270 degrees
- moved C3 95.0 mm to (3.56, 49.3)
- moved S1 94.4 mm to (3.81, 42.9), turned to 90 degrees
- moved C12 87.1 mm to (10.7, 11.4), turned to 90 degrees
- moved C11 86.3 mm to (13.7, 9.65), turned to 180 degrees
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Connections:
- net N$2 renamed DP
- net N$3 renamed DN
- removed net VDDIO: U2.8
- net +3V3: now also C14.1, C5.1, C7.1, C8.1, U2.5, U2.8; no longer C12.1, C6.1, U2.13
- net BATTERY: now also C12.1; no longer C10.1
- net BOARD_POWER: now also C13.1; no longer C11.1
- net GND: now also C13.2, C14.2, U2.2, U2.3, U2.6, U2.7; no longer U2.18
- net HOTFIX_BATT: now also C6.1; no longer C5.1
- net IMU_INT: now also U2.4; no longer U2.12
- net SPI_IMU_CS: now also U2.12; no longer U2.22
- net SPI_MISO: now also U2.1; no longer U2.9
- net SPI_MOSI: now also U2.14; no longer U2.24
- net SPI_SCK: now also U2.13; no longer U2.23
- net VCC: now also C10.1, C11.1; no longer C7.1, C8.1
Routing:
- net MCU_RESET: track 0.00 -> 15.6 mm
- net SPI_MOSI: track 0.00 -> 10.2 mm, vias 0 -> 2
- net SPI_IMU_CS: track 0.00 -> 7.04 mm, vias 0 -> 2
- net SPI_MISO: track 0.00 -> 6.23 mm, vias 0 -> 2
- net IMU_INT: track 0.00 -> 6.22 mm
- net +3V3: track 0.00 -> 3.95 mm
- net SPI_SCK: track 0.00 -> 3.85 mm
- net GPS_DP: track 0.00 -> 2.38 mm
- net GPS_DN: track 0.00 -> 2.38 mm
Other:
- outline, holes or cut-outs redrawn
