File: boards/rev_A/epoch_revA.brd (EAGLE design)
At the start: 38.1 x 50.8 mm, 52 parts, among them J1 Qwiic Right Angle, J2 USB4105-GF-A, U1 ESP32-WROVER-B, U2 BMX160, U3 U-BLOX_NEO-M9N, U4 USBLC6-2P6, U5 MCP73811T-420I/OT, U6 3.3V, Y1 W3011

Commit message: working on rough layout
Parts:
- moved C13 100.0 mm to (57.1, 48.5)
- moved C14 97.0 mm to (53.1, 50.8)
- moved U6 83.7 mm to (57.1, 41.9)
- moved R5 76.5 mm to (31.2, 33.3)
- moved JP1 75.9 mm to (35.3, 36.8), turned to 90 degrees
- moved C2 68.4 mm to (32.5, 44.7), turned to 90 degrees
- moved J1 58.8 mm to (5.33, 17.8), turned to 270 degrees
- moved J3 56.5 mm to (47.2, 45.7), turned to 270 degrees
- moved R8 55.1 mm to (31.2, 38.1)
- moved S2 54.2 mm to (35.3, 48.8), turned to 180 degrees
- moved R7 52.2 mm to (31.2, 30.2)
- moved R6 52.0 mm to (31.2, 31.8)
- moved R4 47.8 mm to (4.32, 26.7), turned to 90 degrees
- moved LOGO1 47.5 mm to (3.05, 2.03)
- moved J2 46.2 mm to (48.3, 31.8), turned to 90 degrees
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Routing:
- net GPS_DP: track 2.38 -> 0.00 mm
- net GPS_DN: track 2.38 -> 0.00 mm
Other:
- board size 38.1 x 50.8 mm -> 50.8 x 50.8 mm
